File: emu-iv/ERM24064-adapter-direct/ERM24064-adapter.kicad_pcb (KiCad board)
At the start: 2 copper layers, 28.2 x 45.1 mm, 4 parts, among them J1 ERM24064-1-display, J2 ERM24064-1-mainboard

Commit message: correction wrt. to the current limiting resistor for the backlight led.
Connections:
- RV2 pad 2: Net-(RV2-Pad2) -> LED_A
Routing:
- net LED_A: track 18.5 -> 29.5 mm
- net LED_K: track 10.7 -> 1.91 mm
- net Net-(J1-Pad4): vias 0 -> 2
