File: emu-iv/ERM24064-adapter-direct/ERM24064-adapter.sch (KiCad schematic (older format))
At the start: 4 parts, among them J1 ERM24064-1-display, J2 ERM24064-1-mainboard

Commit message: correction wrt. to the current limiting resistor for the backlight led.
Connections:
- net LED_A: now also RV2.2
- no-connect marks 1 -> 0
Other:
- moved on the sheet: RV2
Changed lines of the file:
@@
 L Device:R_POT_TRIM RV2
 U 1 1 60F41176
-P 2900 3250
-F 0 "RV2" H 2830 3204 50  0000 R CNN
-F 1 "Trimpot 1k" H 2830 3295 50  0000 R CNN
-F 2 "Potentiometer_THT:Potentiometer_ACP_CA9-V10_Vertical" H 2900 3250 50  0001 C CNN
-F 3 "~" H 2900 3250 50  0001 C CNN
-	1    2900 3250
+P 3100 3250
+F 0 "RV2" H 3030 3204 50  0000 R CNN
+F 1 "Trimpot 1k" H 3030 3295 50  0000 R CNN
+F 2 "Potentiometer_THT:Potentiometer_ACP_CA9-V10_Vertical" H 3100 3250 50  0001 C CNN
+F 3 "~" H 3100 3250 50  0001 C CNN
+	1    3100 3250
 	-1   0    0    1
 $EndComp
-NoConn ~ 2750 3250
-Text GLabel 2900 3050 1    50   Input ~ 0
+Text GLabel 2850 3250 0    50   Input ~ 0
 LED_A
-Text GLabel 2650 3350 1    50   Input ~ 0
+Text GLabel 2550 3700 1    50   Input ~ 0
 LED_K
 Wire Wire Line
-	2900 3700 2900 3400
-Wire Wire Line
-	2900 3100 2900 3050
+	3100 3700 3100 3400
 Text GLabel 1650 3200 0    50   Input ~ 0
 LED_A
@@
 L power:GND #PWR?
 U 1 1 60F09A85
-P 2650 3350
-F 0 "#PWR?" H 2650 3100 50  0001 C CNN
-F 1 "GND" V 2655 3222 50  0000 R CNN
-F 2 "" H 2650 3350 50  0001 C CNN
-F 3 "" H 2650 3350 50  0001 C CNN
-	1    2650 3350
+P 2550 3700
+F 0 "#PWR?" H 2550 3450 50  0001 C CNN
+F 1 "GND" V 2555 3572 50  0000 R CNN
+F 2 "" H 2550 3700 50  0001 C CNN
+F 3 "" H 2550 3700 50  0001 C CNN
+	1    2550 3700
 	1    0    0    -1
 $EndComp
@@
 L power:+5V #PWR?
 U 1 1 60F0B33E
-P 2900 3700
-F 0 "#PWR?" H 2900 3550 50  0001 C CNN
-F 1 "+5V" V 2915 3828 50  0000 L CNN
-F 2 "" H 2900 3700 50  0001 C CNN
-F 3 "" H 2900 3700 50  0001 C CNN
-	1    2900 3700
+P 3100 3700
+F 0 "#PWR?" H 3100 3550 50  0001 C CNN
+F 1 "+5V" V 3115 3828 50  0000 L CNN
+F 2 "" H 3100 3700 50  0001 C CNN
+F 3 "" H 3100 3700 50  0001 C CNN
+	1    3100 3700
 	-1   0    0    1
 $EndComp
+Wire Wire Line
+	2850 3250 2900 3250
+Wire Wire Line
+	2900 3250 2900 2950
+Wire Wire Line
+	2900 2950 3100 2950
+Wire Wire Line
+	3100 2950 3100 3100
+Connection ~ 2900 3250
+Wire Wire Line
+	2900 3250 2950 3250
 $EndSCHEMATC
